File: pcb/main/power_supply.sch (KiCad schematic (older format))
At the start: 11 parts, among them J5 Conn_02x02_Odd_Even, J6 Conn_02x02_Odd_Even, J7 Conn_02x02_Odd_Even, U2 LP3990MF-3.3_NOPB

Commit message: Finished PCB layout
Changed lines of the file:
@@
 F 3 "~" H 7150 3900 50  0001 C CNN
 	1    7150 3900
-	1    0    0    -1
+	-1   0    0    -1
 $EndComp
 $Comp
